File: PCB/hackpad.kicad_pcb (KiCad board)
At the start: 2 copper layers, 82.4 x 57.2 mm, 10 parts, among them J1 OLED_DISPLAY, SW1 SW_Push, SW2 SW_Push, SW3 SW_Push, SW4 SW_Push, SW5 SW_Push, SW6 SW_Push, U1 XIAO-RP2040-DIP

Commit message: Revision 2V
Parts:
- D1, D2: value SK6812MINI -> SK6812
- moved D2 1.87 mm to (132.6, 86.0)
- moved D1 1.51 mm to (121.8, 85.8)
- moved J1 0.05 mm to (68.8, 38.9)
Connections:
- D1 pad 1: Net-(D1-DOUT) -> GND
- D1 pad 2: GND -> Net-(D1-DIN)
- D1 pad 3: Net-(D1-DIN) -> +5V
- D1 pad 4: +5V -> Net-(D1-DOUT)
- D2 pad 1: unconnected-(D2-DOUT-Pad1) -> GND
- D2 pad 2: GND -> Net-(D1-DOUT)
- D2 pad 3: Net-(D1-DOUT) -> +5V
- D2 pad 4: +5V -> unconnected-(D2-DOUT-Pad4)
- J1 pad 1: +5V -> GND
- J1 pad 2: GND -> +3.3V
- U1 pad 12: unconnected-(U1-3V3-Pad12) -> +3.3V
- U1 pad 14: +5V -> unconnected-(U1-VBUS-Pad14)_1
Routing:
- net +3.3V: track 0.00 -> 69.8 mm
- net +5V: track 80.2 -> 11.5 mm, vias 2 -> 0
- net Net-(U1-GPIO4/MISO): track 87.7 -> 50.6 mm, vias 0 -> 1
- net Net-(U1-GPIO26/ADC0/A0): track 35.4 -> 58.4 mm, vias 1 -> 0
- net Net-(U1-GPIO1/RX): track 75.7 -> 62.3 mm, vias 0 -> 1
- net Net-(U1-GPIO0/TX): track 35.2 -> 23.6 mm
- net Net-(D1-DOUT): track 19.3 -> 8.11 mm
- net SCL: track 35.5 -> 24.7 mm
- net GND: track 187.3 -> 195.4 mm
- net Net-(D1-DIN): track 27.6 -> 33.7 mm, vias 1 -> 0
- net Net-(U1-GPIO3/MOSI): track 49.4 -> 46.1 mm, vias 1 -> 0
