File: PCB/hackpad.kicad_sch (KiCad schematic)
At the start: 10 parts, among them J1 OLED_DISPLAY, SW1 SW_Push, SW2 SW_Push, SW3 SW_Push, SW4 SW_Push, SW5 SW_Push, SW6 SW_Push, U1 XIAO-RP2040-DIP

Commit message: Revision 2V
Parts:
- removed D1, D2: SK6812MINI, LED_SMD:LED_SK6812MINI_PLCC4_3.5x3.5mm_P1.75mm, symbol LED:SK6812MINI
- added D1, D2: SK6812, LED_SMD:LED_SK6812MINI_PLCC4_3.5x3.5mm_P1.75mm, symbol LED:SK6812
Connections:
- net +5V: now also D1.3 (VDD), D2.3 (VDD); no longer J1.1 (Pin_1), U1.14 (VBUS)
- net GND: now also J1.1 (Pin_1), D1.1 (VSS), D2.1 (VSS); no longer J1.2 (Pin_2)
- net +3.3V: now reaches U1.12 (3V3)
- net +3.3V: now also J1.2 (Pin_2)
- net at U1.2 (GPIO27/ADC1/A1): now also D1.2 (DIN)
- new net: D1.4 (DOUT), D2.2 (DIN)
- no-connect marks 0 -> 4
